Commit message: updated files

File: src/campero_common/campero_description/urdf/robotiq_c2/robotiq_85_gripper.transmission.xacro (robot description, xacro)
@@ -1,48 +1,42 @@
 <?xml version="1.0"?>
-<robot xmlns:xacro="http://wiki.ros.org/xacro">
+<robot xmlns:xacro="http://www.ros.org/wiki/xacro">
   <xacro:macro name="robotiq_85_gripper_transmission" params="prefix">
-        <transmission name="${prefix}robotiq_85_left_knuckle_trans">
-            <type>transmission_interface/SimpleTransmission</type>
-            <joint name="${prefix}robotiq_85_left_knuckle_joint">
-                <hardwareInterface>hardware_interface/PositionJointInterface</hardwareInterface>
-            </joint>
-            <actuator name="${prefix}robotiq_85_left_knuckle_motor">
-                <mechanicalReduction>1</mechanicalReduction>
-                <hardwareInterface>hardware_interface/PositionJointInterface</hardwareInterface>
-            </actuator>
-        </transmission>
-        <gazebo>
-                <!-- loading plugin: mimic joints works in gazebo now -->
-            <plugin filename="libroboticsgroup_gazebo_mimic_joint_plugin.so" name="${prefix}mimic_robotiq_85_1">
-                <joint>${prefix}robotiq_85_left_knuckle_joint</joint>
-                <mimicJoint>${prefix}robotiq_85_right_knuckle_joint</mimicJoint>
-                <!--multiplier>1.0</multiplier>
-                <offset>0.0</offset-->
-            </plugin>
-            <plugin filename="libroboticsgroup_gazebo_mimic_joint_plugin.so" name="${prefix}mimic_robotiq_85_2">
-                <joint>${prefix}robotiq_85_left_knuckle_joint</joint>
-                <mimicJoint>${prefix}robotiq_85_left_inner_knuckle_joint</mimicJoint>
-                <!--multiplier>1.0</multiplier>
-                <offset>0.0</offset-->
-            </plugin>
-            <plugin filename="libroboticsgroup_gazebo_mimic_joint_plugin.so" name="${prefix}mimic_robotiq_85_3">
-                <joint>${prefix}robotiq_85_left_knuckle_joint</joint>
-                <mimicJoint>${prefix}robotiq_85_right_inner_knuckle_joint</mimicJoint>
-                <!--multiplier>1.0</multiplier>
-                <offset>0.0</offset-->
-            </plugin>
-            <plugin filename="libroboticsgroup_gazebo_mimic_joint_plugin.so" name="${prefix}mimic_robotiq_85_4">
-                <joint>${prefix}robotiq_85_left_knuckle_joint</joint>
-                <mimicJoint>${prefix}robotiq_85_left_finger_tip_joint</mimicJoint>
-                <multiplier>-1.0</multiplier>
-                <offset>0.0</offset>
-            </plugin>
-            <plugin filename="libroboticsgroup_gazebo_mimic_joint_plugin.so" name="${prefix}mimic_robotiq_85_5">
-                <joint>${prefix}robotiq_85_left_knuckle_joint</joint>
-                <mimicJoint>${prefix}robotiq_85_right_finger_tip_joint</mimicJoint>
-                <multiplier>-1.0</multiplier>
-                <offset>0.0</offset>
-            </plugin>
-        </gazebo>
-    </xacro:macro>
+    <transmission name="${prefix}robotiq_85_left_knuckle_trans">
+      <type>transmission_interface/SimpleTransmission</type>
+      <joint name="${prefix}robotiq_85_left_knuckle_joint">
+        <hardwareInterface>hardware_interface/PositionJointInterface</hardwareInterface>
+      </joint>
+      <actuator name="${prefix}robotiq_85_left_knuckle_motor">
+        <mechanicalReduction>1</mechanicalReduction>
+        <hardwareInterface>hardware_interface/PositionJointInterface</hardwareInterface>
+      </actuator>
+    </transmission>
+    <!-- Mimic joints -->
+    <gazebo>
+      <plugin filename="libgazebo_mimic_joint_plugin.so" name="${prefix}mimic_robotiq_85_1">
+        <joint>${prefix}robotiq_85_left_knuckle_joint</joint>
+        <mimicJoint>${prefix}robotiq_85_right_knuckle_joint</mimicJoint>
+      </plugin>
+      <plugin filename="libgazebo_mimic_joint_plugin.so" name="${prefix}mimic_robotiq_85_2">
+        <joint>${prefix}robotiq_85_left_knuckle_joint</joint>
+        <mimicJoint>${prefix}robotiq_85_left_inner_knuckle_joint</mimicJoint>
+      </plugin>
+      <plugin filename="libgazebo_mimic_joint_plugin.so" name="${prefix}mimic_robotiq_85_3">
+        <joint>${prefix}robotiq_85_left_knuckle_joint</joint>
+        <mimicJoint>${prefix}robotiq_85_right_inner_knuckle_joint</mimicJoint>
+      </plugin>
+      <plugin filename="libgazebo_mimic_joint_plugin.so" name="${prefix}mimic_robotiq_85_4">
+        <joint>${prefix}robotiq_85_left_knuckle_joint</joint>
+        <mimicJoint>${prefix}robotiq_85_left_finger_tip_joint</mimicJoint>
+        <multiplier>-1.0</multiplier>
+        <offset>0.0</offset>
+      </plugin>
+      <plugin filename="libgazebo_mimic_joint_plugin.so" name="${prefix}mimic_robotiq_85_5">
+        <joint>${prefix}robotiq_85_left_knuckle_joint</joint>
+        <mimicJoint>${prefix}robotiq_85_right_finger_tip_joint</mimicJoint>
+        <multiplier>-1.0</multiplier>
+        <offset>0.0</offset>
+      </plugin>
+    </gazebo>
+  </xacro:macro>
 </robot>

File: src/campero_robot_real/campero_robot_real_description/urdf/campero_lm.urdf.xacro (robot description, xacro)
@@ -16,5 +16,5 @@
 	<xacro:property name="PI" value="3.1415926535897931"/>
 	<!-- Include gripper description -->
-	<xacro:include filename="$(find campero_description)/urdf/robotiq_c2/robotiq_85_gripper.urdf.xacro" />
+    <xacro:include filename="$(find campero_description)/urdf/robotiq_c2/robotiq_85_gripper.urdf.xacro" />
 	<!-- Include force sensor description -->
 	<xacro:include filename="$(find campero_description)/urdf/robotiq_force_torque_sensor/robotiq_fts300.urdf.xacro" />
@@ -113,4 +113,15 @@
 				<origin xyz="${gps_offset_x} ${gps_offset_y} ${gps_offset_z}"/>
 		</xacro:sensor_gps-->
+		<!-- UR-10 ARM -->
+		<xacro:arg name="kinematics_config" default="$(find campero_robot_real_bring_up)/config/campero_ur10_calibration.yaml"/>
+		<xacro:ur10_robot prefix="$(arg prefix)ur10_" joint_limited="true"
+			shoulder_pan_lower_limit="${-2*PI}" shoulder_pan_upper_limit="${2*PI}"
+    		shoulder_lift_lower_limit="${-PI}" shoulder_lift_upper_limit="${0}"
+    		elbow_joint_lower_limit="${-PI}" elbow_joint_upper_limit="${PI}"
+    		wrist_1_lower_limit="${-PI}" wrist_1_upper_limit="${PI}"
+    		wrist_2_lower_limit="${-PI}" wrist_2_upper_limit="${PI}"
+    		wrist_3_lower_limit="${-PI}" wrist_3_upper_limit="${PI}"
+			kinematics_file="${load_yaml('$(arg kinematics_config)')}">
+		</xacro:ur10_robot>
 		<!--Unimos el brazo con la base del campero-->
 		<joint name="$(arg prefix)ur10_arm_base_joint" type="fixed">
@@ -127,15 +138,4 @@
 			<origin xyz="0 0.0 0" rpy="0 -1.57 0"/>
 		</xacro:robotiq_85_gripper>
-		<!-- UR-10 ARM -->
-		<xacro:arg name="kinematics_config" default="$(find campero_robot_real_bring_up)/config/campero_ur10_calibration.yaml"/>
-		<xacro:ur10_robot prefix="$(arg prefix)ur10_" joint_limited="true"
-			shoulder_pan_lower_limit="${-2*PI}" shoulder_pan_upper_limit="${2*PI}"
-    		shoulder_lift_lower_limit="${-PI}" shoulder_lift_upper_limit="${0}"
-    		elbow_joint_lower_limit="${-PI}" elbow_joint_upper_limit="${PI}"
-    		wrist_1_lower_limit="${-PI}" wrist_1_upper_limit="${PI}"
-    		wrist_2_lower_limit="${-PI}" wrist_2_upper_limit="${PI}"
-    		wrist_3_lower_limit="${-PI}" wrist_3_upper_limit="${PI}"
-			kinematics_file="${load_yaml('$(arg kinematics_config)')}">
-		</xacro:ur10_robot>
    </xacro:macro>
    <xacro:ros_control/>
